Commit message: multi robot works

File: main_simulation/urdf/ur3.urdf.xacro (robot description, xacro)
@@ -90,5 +90,5 @@
      trajectory_port="$(arg trajectory_port)"
      >
-     <origin xyz="2 2 2" rpy="3.14159 0 3.14159" />          <!-- position robot in the world -->
+     <origin xyz="1 1 1" rpy="3.14159 0 3.14159" />          <!-- position robot in the world -->
    </xacro:ur_robot>
      <!-- Gripper -->
@@ -103,7 +103,10 @@
     </gazebo>
     <gazebo>
-      <plugin filename="libgazebo_ros2_control.so" name="gazebo_ros2_control">
+      <plugin filename="libgazebo_ros2_control.so" name="gazebo_ros2_control_robot2">
+        <!-- <controller_manager_node_name>/robot2/controller_manager</controller_manager_node_name> -->
+        <controller_manager_prefix_node_name>/robot2</controller_manager_prefix_node_name>
+        <parameters>$(find main_simulation)/config/ur3_controllers.yaml</parameters>
         <ros>
-          <namespace>/robot2</namespace>
+          <namespace>robot2</namespace>
           <remapping>/tf:=/robot2/tf</remapping>
         </ros>

File: main_simulation/urdf/ur5.urdf.xacro (robot description, xacro)
@@ -103,7 +103,10 @@
     </gazebo>
     <gazebo>
-      <plugin filename="libgazebo_ros2_control.so" name="gazebo_ros2_control">
+      <plugin filename="libgazebo_ros2_control.so" name="gazebo_ros2_control_robot1">
+        <parameters>$(find main_simulation)/config/ur5_controllers.yaml</parameters>
+        <controller_manager_prefix_node_name>/robot1</controller_manager_prefix_node_name>
+        <!-- <controller_manager_node_name>/robot1/controller_manager</controller_manager_node_name> -->
         <ros>
-          <namespace>/robot1</namespace>
+          <namespace>robot1</namespace>
           <remapping>/tf:=/robot1/tf</remapping>
         </ros>

Commit message: commit generico

File: main_simulation/urdf/ur3.urdf.xacro (robot description, xacro)
@@ -90,5 +90,6 @@
      trajectory_port="$(arg trajectory_port)"
      >
-     <origin xyz="1 1 1" rpy="3.14159 0 3.14159" />          <!-- position robot in the world -->
+     <origin xyz="0 0.61 0.88" rpy="0 0 1.570795" />          <!-- position robot in the world -->
+     <!-- <origin xyz="0 0 1.79" rpy="3.14159 0 3.14159" />          position robot in the world -->
    </xacro:ur_robot>
      <!-- Gripper -->

Commit message: working on real robots

File: main_simulation/urdf/ur3.urdf.xacro (robot description, xacro)
@@ -1,103 +1,114 @@
 <?xml version="1.0"?>
 <robot xmlns:xacro="http://wiki.ros.org/xacro" name="$(arg name)">
-   <!-- robot name parameter -->
-   <xacro:arg name="name" default="ur"/>
-   <!-- import main macro -->
-   <xacro:include filename="$(find ur_description)/urdf/ur_macro.xacro"/>
-   <xacro:include filename="$(find gripper_description)/urdf/soft_robotics_gripper.xacro"/>
-   <!-- possible 'ur_type' values: ur3, ur3e, ur5, ur5e, ur10, ur10e, ur16e, ur20, ur30 -->
-   <!-- the default value should raise an error in case this was called without defining the type -->
-   <xacro:arg name="ur_type" default="ur5e"/>
-   <!-- parameters -->
-   <xacro:arg name="tf_prefix" default="" />
-   <xacro:arg name="joint_limit_params" default="$(find ur_description)/config/$(arg ur_type)/joint_limits.yaml"/>
-   <xacro:arg name="kinematics_params" default="$(find ur_description)/config/$(arg ur_type)/default_kinematics.yaml"/>
-   <xacro:arg name="physical_params" default="$(find ur_description)/config/$(arg ur_type)/physical_parameters.yaml"/>
-   <xacro:arg name="visual_params" default="$(find ur_description)/config/$(arg ur_type)/visual_parameters.yaml"/>
-   <xacro:arg name="transmission_hw_interface" default=""/>
-   <xacro:arg name="safety_limits" default="false"/>
-   <xacro:arg name="safety_pos_margin" default="0.15"/>
-   <xacro:arg name="safety_k_position" default="20"/>
-   <!-- ros2_control related parameters -->
-   <xacro:arg name="headless_mode" default="true" />
-   <xacro:arg name="robot_ip" default="0.0.0.0" />
-   <xacro:arg name="script_filename" default=""/>
-   <xacro:arg name="output_recipe_filename" default=""/>
-   <xacro:arg name="input_recipe_filename" default=""/>
-   <xacro:arg name="reverse_ip" default="0.0.0.0"/>
-   <xacro:arg name="script_command_port" default="50004"/>
-   <xacro:arg name="reverse_port" default="50001"/>
-   <xacro:arg name="script_sender_port" default="50002"/>
-   <xacro:arg name="trajectory_port" default="50003"/>
-   <!--   tool communication related parameters-->
-   <xacro:arg name="use_tool_communication" default="false" />
-   <xacro:arg name="tool_voltage" default="0" />
-   <xacro:arg name="tool_parity" default="0" />
-   <xacro:arg name="tool_baud_rate" default="115200" />
-   <xacro:arg name="tool_stop_bits" default="1" />
-   <xacro:arg name="tool_rx_idle_chars" default="1.5" />
-   <xacro:arg name="tool_tx_idle_chars" default="3.5" />
-   <xacro:arg name="tool_device_name" default="/tmp/ttyUR" />
-   <xacro:arg name="tool_tcp_port" default="54321" />
-     <!-- Simulation parameters -->
-   <xacro:arg name="use_fake_hardware" default="false" />
-   <xacro:arg name="fake_sensor_commands" default="false" />
-   <xacro:arg name="sim_gazebo" default="false" />
-   <xacro:arg name="sim_ignition" default="false" />
-   <xacro:arg name="simulation_controllers" default="" />
-   <!-- initial position for simulations (Fake Hardware, Gazebo, Ignition) -->
-   <xacro:arg name="initial_positions_file" default="$(find main_simulation)/config/initial_positions.yaml"/>
-   <!-- convert to property to use substitution in function -->
-   <xacro:property name="initial_positions_file" default="$(arg initial_positions_file)"/>
-   <!-- create link fixed to the "world" -->
-   <link name="world" />
-   <!-- arm -->
-   <xacro:ur_robot
-     name="$(arg name)"
-     tf_prefix="$(arg tf_prefix)"
-     parent="world"
-     joint_limits_parameters_file="$(arg joint_limit_params)"
-     kinematics_parameters_file="$(arg kinematics_params)"
-     physical_parameters_file="$(arg physical_params)"
-     visual_parameters_file="$(arg visual_params)"
-     transmission_hw_interface="$(arg transmission_hw_interface)"
-     safety_limits="$(arg safety_limits)"
-     safety_pos_margin="$(arg safety_pos_margin)"
-     safety_k_position="$(arg safety_k_position)"
-     use_fake_hardware="$(arg use_fake_hardware)"
-     fake_sensor_commands="$(arg fake_sensor_commands)"
-     sim_gazebo="$(arg sim_gazebo)"
-     sim_ignition="$(arg sim_ignition)"
-     headless_mode="$(arg headless_mode)"
-     initial_positions="${xacro.load_yaml(initial_positions_file)}"
-     use_tool_communication="$(arg use_tool_communication)"
-     tool_voltage="$(arg tool_voltage)"
-     tool_parity="$(arg tool_parity)"
-     tool_baud_rate="$(arg tool_baud_rate)"
-     tool_stop_bits="$(arg tool_stop_bits)"
-     tool_rx_idle_chars="$(arg tool_rx_idle_chars)"
-     tool_tx_idle_chars="$(arg tool_tx_idle_chars)"
-     tool_device_name="$(arg tool_device_name)"
-     tool_tcp_port="$(arg tool_tcp_port)"
-     robot_ip="$(arg robot_ip)"
-     script_filename="$(arg script_filename)"
-     output_recipe_filename="$(arg output_recipe_filename)"
-     input_recipe_filename="$(arg input_recipe_filename)"
-     reverse_ip="$(arg reverse_ip)"
-     script_command_port="$(arg script_command_port)"
-     reverse_port="$(arg reverse_port)"
-     script_sender_port="$(arg script_sender_port)"
-     trajectory_port="$(arg trajectory_port)"
-     >
-     <origin xyz="0 0.61 0.88" rpy="0 0 1.570795" />          <!-- position robot in the world -->
-     <!-- <origin xyz="0 0 1.79" rpy="3.14159 0 3.14159" />          position robot in the world -->
-   </xacro:ur_robot>
-     <!-- Gripper -->
-   <xacro:soft_robotics_gripper
+  <!-- robot name parameter -->
+  <xacro:arg name="name" default="ur" />
+  <!-- import main macro -->
+  <xacro:include filename="$(find ur_description)/urdf/ur_macro.xacro" />
+  <xacro:include filename="$(find robotiq_description)/urdf/robotiq_2f_85_macro.urdf.xacro" />
+  <xacro:include filename="$(find gripper_description)/urdf/soft_robotics_gripper.xacro" />
+  <!-- possible 'ur_type' values: ur3, ur3e, ur5, ur5e, ur10, ur10e, ur16e, ur20, ur30 -->
+  <!-- the default value should raise an error in case this was called without defining the type -->
+  <xacro:arg name="ur_type" default="ur5e" />
+  <!-- parameters -->
+  <xacro:arg name="tf_prefix" default="" />
+  <xacro:arg name="joint_limit_params"
+    default="$(find ur_description)/config/$(arg ur_type)/joint_limits.yaml" />
+  <xacro:arg name="kinematics_params"
+    default="$(find ur_description)/config/$(arg ur_type)/default_kinematics.yaml" />
+  <xacro:arg name="physical_params"
+    default="$(find ur_description)/config/$(arg ur_type)/physical_parameters.yaml" />
+  <xacro:arg name="visual_params"
+    default="$(find ur_description)/config/$(arg ur_type)/visual_parameters.yaml" />
+  <xacro:arg name="transmission_hw_interface" default="" />
+  <xacro:arg name="safety_limits" default="false" />
+  <xacro:arg name="safety_pos_margin" default="0.15" />
+  <xacro:arg name="safety_k_position" default="20" />
+  <!-- ros2_control related parameters -->
+  <xacro:arg name="headless_mode" default="true" />
+  <xacro:arg name="robot_ip" default="0.0.0.0" />
+  <xacro:arg name="script_filename" default="" />
+  <xacro:arg name="output_recipe_filename" default="" />
+  <xacro:arg name="input_recipe_filename" default="" />
+  <xacro:arg name="reverse_ip" default="0.0.0.0" />
+  <xacro:arg name="script_command_port" default="50004" />
+  <xacro:arg name="reverse_port" default="50001" />
+  <xacro:arg name="script_sender_port" default="50002" />
+  <xacro:arg name="trajectory_port" default="50003" />
+  <!--   tool communication related parameters-->
+  <xacro:arg name="use_tool_communication" default="false" />
+  <xacro:arg name="tool_voltage" default="0" />
+  <xacro:arg name="tool_parity" default="0" />
+  <xacro:arg name="tool_baud_rate" default="115200" />
+  <xacro:arg name="tool_stop_bits" default="1" />
+  <xacro:arg name="tool_rx_idle_chars" default="1.5" />
+  <xacro:arg name="tool_tx_idle_chars" default="3.5" />
+  <xacro:arg name="tool_device_name" default="/tmp/ttyUR" />
+  <xacro:arg name="tool_tcp_port" default="54321" />
+  <!-- Simulation parameters -->
+  <xacro:arg name="use_fake_hardware" default="false" />
+  <xacro:arg name="fake_sensor_commands" default="false" />
+  <xacro:arg name="sim_gazebo" default="false" />
+  <xacro:arg name="sim_ignition" default="false" />
+  <xacro:arg name="simulation_controllers" default="" />
+  <!-- initial position for simulations (Fake Hardware, Gazebo, Ignition) -->
+  <xacro:arg name="initial_positions_file"
+    default="$(find main_simulation)/config/initial_positions_ur3.yaml" />
+  <!-- convert to property to use substitution in function -->
+  <xacro:property name="initial_positions_file" default="$(arg initial_positions_file)" />
+  <!-- create link fixed to the "world" -->
+  <link name="world" />
+  <!-- arm -->
+  <xacro:ur_robot
+    name="$(arg name)"
+    tf_prefix="$(arg tf_prefix)"
+    parent="world"
+    joint_limits_parameters_file="$(arg joint_limit_params)"
+    kinematics_parameters_file="$(arg kinematics_params)"
+    physical_parameters_file="$(arg physical_params)"
+    visual_parameters_file="$(arg visual_params)"
+    transmission_hw_interface="$(arg transmission_hw_interface)"
+    safety_limits="$(arg safety_limits)"
+    safety_pos_margin="$(arg safety_pos_margin)"
+    safety_k_position="$(arg safety_k_position)"
+    use_fake_hardware="$(arg use_fake_hardware)"
+    fake_sensor_commands="$(arg fake_sensor_commands)"
+    sim_gazebo="$(arg sim_gazebo)"
+    sim_ignition="$(arg sim_ignition)"
+    headless_mode="$(arg headless_mode)"
+    initial_positions="${xacro.load_yaml(initial_positions_file)}"
+    use_tool_communication="$(arg use_tool_communication)"
+    tool_voltage="$(arg tool_voltage)"
+    tool_parity="$(arg tool_parity)"
+    tool_baud_rate="$(arg tool_baud_rate)"
+    tool_stop_bits="$(arg tool_stop_bits)"
+    tool_rx_idle_chars="$(arg tool_rx_idle_chars)"
+    tool_tx_idle_chars="$(arg tool_tx_idle_chars)"
+    tool_device_name="$(arg tool_device_name)"
+    tool_tcp_port="$(arg tool_tcp_port)"
+    robot_ip="$(arg robot_ip)"
+    script_filename="$(arg script_filename)"
+    output_recipe_filename="$(arg output_recipe_filename)"
+    input_recipe_filename="$(arg input_recipe_filename)"
+    reverse_ip="$(arg reverse_ip)"
+    script_command_port="$(arg script_command_port)"
+    reverse_port="$(arg reverse_port)"
+    script_sender_port="$(arg script_sender_port)"
+    trajectory_port="$(arg trajectory_port)"
+  >
+    <!-- <origin xyz="0 0.61 0.88" rpy="0 0 1.570795" />          position robot in the world -->
+    <origin xyz="0 0.61 1.88" rpy="0 0 1.570795" />          <!-- position robot in the world -->
+    <!-- <origin xyz="0 0 1.79" rpy="3.14159 0 3.14159" />          position robot in the world -->
+  </xacro:ur_robot>
+  <!-- Gripper -->
+  <!-- <xacro:soft_robotics_gripper
     prefix="$(arg tf_prefix)"
     parent="$(arg tf_prefix)flange">
-    <origin xyz="0 0 0" rpy="0 0 0"/>
-   </xacro:soft_robotics_gripper>
-   <xacro:if value="$(arg sim_gazebo)">
+    <origin xyz="0 0 0" rpy="0 0 0" />
+  </xacro:soft_robotics_gripper> -->
+  <xacro:robotiq_gripper name="RobotiqGripperHardwareInterface" prefix="$(arg tf_prefix)"
+    parent="$(arg tf_prefix)flange" use_fake_hardware="false">
+    <origin xyz="0 0 0" rpy="0 1.57 0" />
+  </xacro:robotiq_gripper>
+  <xacro:if value="$(arg sim_gazebo)">
     <!-- Gazebo plugins -->
     <gazebo reference="world">
@@ -106,5 +117,6 @@
       <plugin filename="libgazebo_ros2_control.so" name="gazebo_ros2_control_robot2">
         <!-- <controller_manager_node_name>/robot2/controller_manager</controller_manager_node_name> -->
-        <controller_manager_prefix_node_name>/robot2</controller_manager_prefix_node_name>
+        <!-- <controller_manager_prefix_node_name>/robot2</controller_manager_prefix_node_name> -->
+        <robot_param_node>/robot2/robot_state_publisher</robot_param_node>
         <parameters>$(find main_simulation)/config/ur3_controllers.yaml</parameters>
         <ros>
@@ -112,14 +124,15 @@
           <!-- <remapping>/tf:=/robot2/tf</remapping> -->
         </ros>
-        <parameters>$(arg simulation_controllers)</parameters>
+        <!-- <parameters>$(arg simulation_controllers)</parameters> -->
       </plugin>
     </gazebo>
   </xacro:if>
   <!-- <xacro:if value="$(arg sim_ignition)"> -->
-    <!-- Gazebo plugins -->
-    <!-- <gazebo reference="world">
+  <!-- Gazebo plugins -->
+  <!-- <gazebo reference="world">
     </gazebo>
     <gazebo>
-      <plugin filename="libign_ros2_control-system.so" name="ign_ros2_control::IgnitionROS2ControlPlugin">
+      <plugin filename="libign_ros2_control-system.so"
+  name="ign_ros2_control::IgnitionROS2ControlPlugin">
         <parameters>$(arg simulation_controllers)</parameters>
         <controller_manager_node_name>$(arg tf_prefix)controller_manager</controller_manager_node_name>
