Commit message: quasi funzionante

File: gripper_description/urdf/soft_robotics_gripper.xacro (robot description, xacro)
@@ -8,10 +8,10 @@
   </material>
   <xacro:macro name="soft_robotics_gripper" params="prefix parent *origin">
-    <joint name="soft_robotics_gripper_base_joint" type="fixed">
+    <joint name="${prefix}soft_robotics_gripper_base_joint" type="fixed">
       <origin xyz="0 0 0" rpy="${pi/2} 0 ${pi/2}" />
       <parent link="${parent}" />
-      <child link="soft_robotics_gripper_base_link" />
+      <child link="${prefix}soft_robotics_gripper_base_link" />
     </joint>
-    <link name="soft_robotics_gripper_base_link">
+    <link name="${prefix}soft_robotics_gripper_base_link">
       <visual>
         <origin rpy="0 0 0" xyz="0 0 -0.0095" />
@@ -33,11 +33,11 @@
       </inertial>
     </link>
-    <joint name="soft_robotics_gripper_left_finger_joint1" type="fixed">
+    <joint name="${prefix}soft_robotics_gripper_left_finger_joint1" type="fixed">
       <origin xyz="0 -0.028 0.09" rpy=" 0 0 0" />
-      <parent link="soft_robotics_gripper_base_link" />
-      <child link="soft_robotics_left_finger_link1" />
+      <parent link="${prefix}soft_robotics_gripper_base_link" />
+      <child link="${prefix}soft_robotics_left_finger_link1" />
       <limit effort="1" velocity="1" lower="-0.30" upper="0" />
     </joint>
-    <link name="soft_robotics_left_finger_link1">
+    <link name="${prefix}soft_robotics_left_finger_link1">
       <visual>
         <origin rpy="0 0 0" xyz="0 0 0" />
@@ -59,11 +59,11 @@
       </inertial>
     </link>
-    <joint name="soft_robotics_gripper_right_finger_joint1" type="fixed">
+    <joint name="${prefix}soft_robotics_gripper_right_finger_joint1" type="fixed">
       <origin xyz="0 0.028 0.09" rpy=" 0 0 ${-pi}" />
-      <parent link="soft_robotics_gripper_base_link" />
-      <child link="soft_robotics_right_finger_link1" />
+      <parent link="${prefix}soft_robotics_gripper_base_link" />
+      <child link="${prefix}soft_robotics_right_finger_link1" />
       <limit effort="1" velocity="1" lower="-0.30" upper="0" />
     </joint>
-    <link name="soft_robotics_right_finger_link1">
+    <link name="${prefix}soft_robotics_right_finger_link1">
       <visual>
         <origin rpy="0 0 0" xyz="0 0 0" />
@@ -85,10 +85,10 @@
       </inertial>
     </link>
-    <joint name="soft_robotics_gripper_left_finger_joint2" type="fixed">
+    <joint name="${prefix}soft_robotics_gripper_left_finger_joint2" type="fixed">
       <origin xyz="0 0.009 0.042" rpy=" 0 0 0" />
-      <parent link="soft_robotics_left_finger_link1" />
-      <child link="soft_robotics_left_finger_link2" />
+      <parent link="${prefix}soft_robotics_left_finger_link1" />
+      <child link="${prefix}soft_robotics_left_finger_link2" />
     </joint>
-    <link name="soft_robotics_left_finger_link2">
+    <link name="${prefix}soft_robotics_left_finger_link2">
       <visual>
         <geometry>
@@ -108,10 +108,10 @@
       </inertial>
     </link>
-    <joint name="soft_robotics_gripper_right_finger_joint2" type="fixed">
+    <joint name="${prefix}soft_robotics_gripper_right_finger_joint2" type="fixed">
       <origin xyz="0 0.009 0.042" rpy=" 0 0 0" />
-      <parent link="soft_robotics_right_finger_link1" />
-      <child link="soft_robotics_right_finger_link2" />
+      <parent link="${prefix}soft_robotics_right_finger_link1" />
+      <child link="${prefix}soft_robotics_right_finger_link2" />
     </joint>
-    <link name="soft_robotics_right_finger_link2">
+    <link name="${prefix}soft_robotics_right_finger_link2">
       <visual>
         <geometry>
@@ -131,32 +131,32 @@
       </inertial>
     </link>
-  <gazebo reference="soft_robotics_gripper_base_link">
+  <gazebo reference="${prefix}soft_robotics_gripper_base_link">
         <material>Gazebo/Grey</material>
   </gazebo>
-  <gazebo reference="soft_robotics_left_finger_link1">
+  <gazebo reference="${prefix}soft_robotics_left_finger_link1">
         <material>Gazebo/Blue</material>
   </gazebo>
-  <gazebo reference="soft_robotics_right_finger_link1">
+  <gazebo reference="${prefix}soft_robotics_right_finger_link1">
         <material>Gazebo/Blue</material>
   </gazebo>
-    <gazebo reference="soft_robotics_left_finger_link2">
+    <gazebo reference="${prefix}soft_robotics_left_finger_link2">
         <material>Gazebo/Blue</material>
   </gazebo>
-  <gazebo reference="soft_robotics_right_finger_link2">
+  <gazebo reference="${prefix}soft_robotics_right_finger_link2">
         <material>Gazebo/Blue</material>
   </gazebo>
     <!-- TRANSMISSION -->
-    <transmission name="right_finger_trans">
+    <transmission name="${prefix}right_finger_trans">
       <type>transmission_interface/SimpleTransmission</type>
-      <joint name="soft_robotics_gripper_left_finger_joint1">
+      <joint name="${prefix}soft_robotics_gripper_left_finger_joint1">
         <hardwareInterface>hardware_interface/PositionJointInterface</hardwareInterface>
       </joint>
-      <actuator name="right_finger_motor">
+      <actuator name="${prefix}right_finger_motor">
         <mechanicalReduction>1</mechanicalReduction>
       </actuator>
     </transmission>
-    <transmission name="left_finger_trans">
+    <transmission name="${prefix}left_finger_trans">
       <type>transmission_interface/SimpleTransmission</type>
-      <joint name="soft_robotics_gripper_right_finger_joint1">
+      <joint name="${prefix}soft_robotics_gripper_right_finger_joint1">
         <hardwareInterface>hardware_interface/PositionJointInterface</hardwareInterface>
       </joint>

File: main_simulation/urdf/ur3.urdf.xacro (robot description, xacro)
@@ -90,5 +90,5 @@
      trajectory_port="$(arg trajectory_port)"
      >
-     <origin xyz="0 0 0" rpy="3.14159 0 3.14159" />          <!-- position robot in the world -->
+     <origin xyz="2 2 2" rpy="3.14159 0 3.14159" />          <!-- position robot in the world -->
    </xacro:ur_robot>
      <!-- Gripper -->
@@ -104,11 +104,15 @@
     <gazebo>
       <plugin filename="libgazebo_ros2_control.so" name="gazebo_ros2_control">
+        <ros>
+          <namespace>/robot2</namespace>
+          <remapping>/tf:=/robot2/tf</remapping>
+        </ros>
         <parameters>$(arg simulation_controllers)</parameters>
       </plugin>
     </gazebo>
   </xacro:if>
-  <xacro:if value="$(arg sim_ignition)">
+  <!-- <xacro:if value="$(arg sim_ignition)"> -->
     <!-- Gazebo plugins -->
-    <gazebo reference="world">
+    <!-- <gazebo reference="world">
     </gazebo>
     <gazebo>
@@ -118,4 +122,4 @@
       </plugin>
     </gazebo>
-  </xacro:if>
+  </xacro:if> -->
 </robot>

File: main_simulation/urdf/ur5.urdf.xacro (robot description, xacro)
@@ -104,11 +104,15 @@
     <gazebo>
       <plugin filename="libgazebo_ros2_control.so" name="gazebo_ros2_control">
+        <ros>
+          <namespace>/robot1</namespace>
+          <remapping>/tf:=/robot1/tf</remapping>
+        </ros>
         <parameters>$(arg simulation_controllers)</parameters>
       </plugin>
     </gazebo>
   </xacro:if>
-  <xacro:if value="$(arg sim_ignition)">
+  <!-- <xacro:if value="$(arg sim_ignition)"> -->
     <!-- Gazebo plugins -->
-    <gazebo reference="world">
+    <!-- <gazebo reference="world">
     </gazebo>
     <gazebo>
@@ -118,4 +122,4 @@
       </plugin>
     </gazebo>
-  </xacro:if>
+  </xacro:if> -->
 </robot>
